File: eagle/old/front-end-eval-boards.sch (EAGLE design)
At the start: 168 parts, among them U1 MAC-24+, U10 TPS6211X, U11 MiniCirc. BPF-A1340+, U12 Qorvo 856930, U13 Murata SF2446E, U2 SI4123, U3 SI4112, U4 QCN-19+, U5 LP38692, U6 TQP3M9036, U7 TQL9092, U8 QPA4463A, U9 TQP7M9106, X1 SMA-142-0701-801/806, X10 SMA-142-0701-801/806, X11 SMA-142-0701-801/806, X12 SMA-142-0701-801/806, X13 SMA-142-0701-801/806, X14 SMA-142-0701-801/806, X15 SMA-142-0701-801/806, X16 SMA, X17 SMA, X18 SMA-142-0701-801/806, X19 SMA-142-0701-801/806, X2 SMA-142-0701-801/806, X20 SMA-142-0701-801/806, X21 SMA-142-0701-801/806, X22 SMA-142-0701-801/806, X23 ECS-TXO-3225, X24 ECS-TXO-3225, X25 SMA-142-0701-801/806, X26 SMA-142-0701-801/806, X27 SMA-142-0701-801/806, X28 SMA-142-0701-801/806, X29 SMA-142-0701-801/806, X3 SMA-142-0701-801/806, X30 SMA-142-0701-801/806, X4 SMA, X5 SMA-142-0701-801/806, X6 SMA-142-0701-801/806, X7 SMA, X8 SMA, X9 SMA

Commit message: Initial Eagle dev boards
Parts:
- added JP29: (no value), pinhead:PINHD-1X2
- added Q1: BSS84, transistor-small-signal:BSS84
- added R21: 47k, rcl:R-US_R0402
Connections:
- new net N$11: JP29.2, Q1.G, R21.1
- new net N$91: JP26.2, Q1.D
- net GND: now also JP29.1
- net N$72: now also Q1.S, R21.2; no longer JP26.2
Other:
- note added: "On/Off Active low"
- moved on the sheet: JP26
Changed lines of the file:
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@@
 <part name="C59" library="rcl" library_urn="urn:adsk.eagle:library:334" deviceset="C-EU" device="C0603" package3d_urn="urn:adsk.eagle:package:23616/2" value="?"/>
 <part name="GND113" library="supply1" library_urn="urn:adsk.eagle:library:371" deviceset="GND" device=""/>
+<part name="Q1" library="transistor-small-signal" library_urn="urn:adsk.eagle:library:401" deviceset="BSS84" device="" package3d_urn="urn:adsk.eagle:package:29752/1"/>
+<part name="JP29" library="pinhead" library_urn="urn:adsk.eagle:library:325" deviceset="PINHD-1X2" device="" package3d_urn="urn:adsk.eagle:package:22435/2"/>
+<part name="GND114" library="supply1" library_urn="urn:adsk.eagle:library:371" deviceset="GND" device=""/>
+<part name="R21" library="rcl" library_urn="urn:adsk.eagle:library:334" deviceset="R-US_" device="R0402" package3d_urn="urn:adsk.eagle:package:23547/3" value="47k"/>
 </parts>
 <sheets>
@@
 <text x="161.29" y="187.96" size="1.778" layer="97" rot="MR180">3.3V
 External</text>
-<text x="161.29" y="123.19" size="1.778" layer="96">2n Trace inductor</text>
+<text x="160.02" y="129.54" size="1.778" layer="96">2n Trace inductor</text>
 <text x="88.9" y="78.74" size="1.778" layer="97">Select Ref</text>
 <text x="58.42" y="55.88" size="1.778" layer="97">16.000 MHz</text>
@@
 <text x="118.11" y="147.32" size="1.778" layer="97">VBias Resistor
 Socket</text>
-<text x="152.4" y="147.32" size="1.778" layer="97">Iref Resistor
+<text x="151.13" y="144.78" size="1.778" layer="97">Iref Resistor
 Socket</text>
 <text x="119.38" y="128.27" size="1.778" layer="97">Inductor?</text>
@@
 <wire x1="68.58" y1="119.38" x2="68.58" y2="100.33" width="0.1524" layer="97" style="shortdash"/>
 <text x="80.01" y="104.14" size="1.778" layer="97">work in progress</text>
-<text x="101.6" y="165.1" size="3.81" layer="97">2W High Linearity Amplifier</text>
-<text x="101.6" y="161.29" size="2.1844" layer="97">26dB Gain @ 436.5 MHz</text>
+<text x="114.3" y="175.26" size="3.81" layer="97">2W High Linearity Amplifier</text>
+<text x="114.3" y="171.45" size="2.1844" layer="97">26dB Gain @ 436.5 MHz</text>
+<text x="77.47" y="153.67" size="1.778" layer="97" align="bottom-right">On/Off
+Active low</text>
 </plain>
 <instances>
@@
 <attribute name="VALUE" x="153.67" y="125.73" size="1.778" layer="96" rot="R90"/>
 </instance>
-<instance part="JP26" gate="A" x="147.32" y="147.32" smashed="yes" rot="R90">
-<attribute name="NAME" x="147.32" y="146.05" size="1.778" layer="95" rot="R180"/>
-<attribute name="VALUE" x="147.32" y="153.035" size="1.778" layer="96" rot="R180"/>
+<instance part="JP26" gate="A" x="147.32" y="144.78" smashed="yes" rot="R90">
+<attribute name="NAME" x="147.32" y="143.51" size="1.778" layer="95" rot="R180"/>
+<attribute name="VALUE" x="147.32" y="150.495" size="1.778" layer="96" rot="R180"/>
 </instance>
 <instance part="D1" gate="G$1" x="132.08" y="139.7" smashed="yes" rot="R180">
@@
 <instance part="GND103" gate="1" x="200.66" y="132.08" smashed="yes">
 <attribute name="VALUE" x="198.12" y="129.54" size="1.778" layer="96"/>
+</instance>
+<instance part="Q1" gate="G$1" x="149.86" y="154.94" smashed="yes">
+<attribute name="NAME" x="152.4" y="154.94" size="1.778" layer="95"/>
+<attribute name="VALUE" x="152.4" y="152.4" size="1.778" layer="96"/>
+</instance>
+<instance part="JP29" gate="G$1" x="80.01" y="157.48" smashed="yes" rot="R180">
+<attribute name="NAME" x="86.36" y="151.765" size="1.778" layer="95" rot="R180"/>
+<attribute name="VALUE" x="86.36" y="162.56" size="1.778" layer="96" rot="R180"/>
+</instance>
+<instance part="GND114" gate="1" x="82.55" y="147.32" smashed="yes">
+<attribute name="VALUE" x="80.01" y="144.78" size="1.778" layer="96"/>
+</instance>
+<instance part="R21" gate="G$1" x="106.68" y="162.56" smashed="yes">
+<attribute name="NAME" x="102.87" y="164.0586" size="1.778" layer="95"/>
+<attribute name="VALUE" x="102.87" y="159.258" size="1.778" layer="96"/>
 </instance>
 </instances>
@@
 <pinref part="C26" gate="G$1" pin="2"/>
 <pinref part="GND103" gate="1" pin="GND"/>
+</segment>
+<segment>
+<pinref part="GND114" gate="1" pin="GND"/>
+<pinref part="JP29" gate="G$1" pin="1"/>
+<wire x1="82.55" y1="149.86" x2="82.55" y2="154.94" width="0.1524" layer="91"/>
 </segment>
 </net>
@@
 <pinref part="JP26" gate="A" pin="1"/>
 <pinref part="L10" gate="G$1" pin="1"/>
-<wire x1="149.86" y1="147.32" x2="149.86" y2="139.7" width="0.1524" layer="91"/>
+<wire x1="149.86" y1="144.78" x2="149.86" y2="139.7" width="0.1524" layer="91"/>
 <wire x1="149.86" y1="139.7" x2="149.86" y2="138.43" width="0.1524" layer="91"/>
 <wire x1="149.86" y1="138.43" x2="149.86" y2="137.16" width="0.1524" layer="91"/>
@@
 <net name="N$72" class="0">
 <segment>
-<pinref part="JP25" gate="A" pin="2"/>
-<wire x1="116.84" y1="149.86" x2="116.84" y2="154.94" width="0.1524" layer="91"/>
-<wire x1="116.84" y1="154.94" x2="149.86" y2="154.94" width="0.1524" layer="91"/>
-<pinref part="JP26" gate="A" pin="2"/>
-<wire x1="149.86" y1="154.94" x2="149.86" y2="149.86" width="0.1524" layer="91"/>
 <pinref part="JP24" gate="G$1" pin="2"/>
 <pinref part="R19" gate="G$1" pin="2"/>
@@
 <wire x1="175.26" y1="154.94" x2="175.26" y2="144.78" width="0.1524" layer="91"/>
 <wire x1="175.26" y1="144.78" x2="175.26" y2="142.24" width="0.1524" layer="91"/>
-<wire x1="149.86" y1="154.94" x2="175.26" y2="154.94" width="0.1524" layer="91"/>
-<junction x="149.86" y="154.94"/>
-<junction x="175.26" y="154.94"/>
 <pinref part="C21" gate="G$1" pin="1"/>
 <wire x1="185.42" y1="142.24" x2="185.42" y2="144.78" width="0.1524" layer="91"/>
@@
 <junction x="200.66" y="144.78"/>
 <junction x="175.26" y="144.78"/>
+<pinref part="Q1" gate="G$1" pin="S"/>
+<wire x1="175.26" y1="162.56" x2="149.86" y2="162.56" width="0.1524" layer="91"/>
+<wire x1="149.86" y1="162.56" x2="149.86" y2="160.02" width="0.1524" layer="91"/>
+<junction x="175.26" y="162.56"/>
+<pinref part="JP25" gate="A" pin="2"/>
+<wire x1="149.86" y1="162.56" x2="116.84" y2="162.56" width="0.1524" layer="91"/>
+<wire x1="116.84" y1="162.56" x2="116.84" y2="149.86" width="0.1524" layer="91"/>
+<junction x="149.86" y="162.56"/>
+<pinref part="R21" gate="G$1" pin="2"/>
+<wire x1="111.76" y1="162.56" x2="116.84" y2="162.56" width="0.1524" layer="91"/>
+<junction x="116.84" y="162.56"/>
 </segment>
 </net>
@@
 </segment>
 </net>
+<net name="N$91" class="0">
+<segment>
+<pinref part="Q1" gate="G$1" pin="D"/>
+<pinref part="JP26" gate="A" pin="2"/>
+<wire x1="149.86" y1="149.86" x2="149.86" y2="147.32" width="0.1524" layer="91"/>
+</segment>
+</net>
+<net name="N$11" class="0">
+<segment>
+<pinref part="Q1" gate="G$1" pin="G"/>
+<pinref part="JP29" gate="G$1" pin="2"/>
+<wire x1="144.78" y1="157.48" x2="109.22" y2="157.48" width="0.1524" layer="91"/>
+<wire x1="109.22" y1="157.48" x2="99.06" y2="157.48" width="0.1524" layer="91"/>
+<pinref part="R21" gate="G$1" pin="1"/>
+<wire x1="99.06" y1="157.48" x2="82.55" y2="157.48" width="0.1524" layer="91"/>
+<wire x1="101.6" y1="162.56" x2="99.06" y2="162.56" width="0.1524" layer="91"/>
+<wire x1="99.06" y1="162.56" x2="99.06" y2="157.48" width="0.1524" layer="91"/>
+<junction x="99.06" y="157.48"/>
+</segment>
+</net>
