File: eagle/amp-LNA-BGB741L7ESD.brd (EAGLE design)
At the start: 25 x 20 mm, 19 parts, among them J1 142-0701-851, J2 142-0701-851, Q1 PMOS, U1 BGB7XXL7ESD

Commit message: BGB741 update values
Parts:
- C6: value 47b -> 47n
- R1: value 2.2k -> 1.5k
Changed lines of the file:
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@@
 <drawing>
 <settings>
-<setting alwaysvectorfont="yes"/>
+<setting alwaysvectorfont="no"/>
 <setting verticaltext="up"/>
 </settings>
@@
 <attribute name="NAME" x="16.1" y="14.2" size="0.3" layer="33" ratio="15" align="center"/>
 </element>
-<element name="C6" library="oresat-rcl" package=".0603-B-NOSILK" value="47b" x="8.6" y="12.6" smashed="yes" rot="R180">
+<element name="C6" library="oresat-rcl" package=".0603-B-NOSILK" value="47n" x="8.6" y="12.6" smashed="yes" rot="R180">
 <attribute name="NAME" x="9.5" y="14.15" size="0.8" layer="25" font="vector" ratio="15" rot="R180"/>
 <attribute name="NAME" x="8.6" y="12.6" size="0.2" layer="33" ratio="15" rot="R180" align="center"/>
@@
 <attribute name="POPULARITY" value="8" x="45.52" y="-15.85" size="1.778" layer="27" display="off"/>
 </element>
-<element name="R1" library="oresat-rcl" package=".0603-B-NOSILK" value="2.2k" x="8.8" y="18.5" smashed="yes" rot="R180">
+<element name="R1" library="oresat-rcl" package=".0603-B-NOSILK" value="1.5k" x="8.8" y="18.5" smashed="yes" rot="R180">
 <attribute name="NAME" x="7.2" y="18.8" size="0.8" layer="25" font="vector" ratio="15" rot="R180"/>
 <attribute name="NAME" x="8.8" y="18.5" size="0.3" layer="33" ratio="15" rot="R180" align="center"/>
