File: eagle/amp-LNA-TQP3M9037.brd (EAGLE design)
At the start: 25 x 20 mm, 18 parts, among them J1 142-0701-851, J2 142-0701-851, U1 TQP3M903X

Commit message: lna-tqp3m9037 update values
Parts:
- R1: value 6.2k -> 5.6k
Changed lines of the file:
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@@
 <attribute name="NAME" x="15.2" y="10.7" size="0.3" layer="33" ratio="15" rot="R270" align="center"/>
 </element>
-<element name="R1" library="oresat-rcl" package=".0603-B-NOSILK" value="6.2k" x="17.3" y="6" smashed="yes">
+<element name="R1" library="oresat-rcl" package=".0603-B-NOSILK" value="5.6k" x="17.3" y="6" smashed="yes">
 <attribute name="NAME" x="18.7" y="5.5" size="0.8" layer="25" font="vector" ratio="15"/>
 <attribute name="NAME" x="17.3" y="6" size="0.3" layer="33" ratio="15" align="center"/>
