File: eagle/quad-hybrid-QCN-xxx+.brd (EAGLE design)
At the start: 20 x 20 mm, 7 parts, among them J1 142-0701-851, J2 142-0701-851, J3 142-0701-851, J4 142-0701-851, U1 QCN-XXX+

Commit message: Update QCN hybrid name
Other:
- board text added: "Quad. Hybrid QCN-XXX+ PSAS / OreSat 2019-11-06 v1 E.M. KJ7AOG"
- board text removed: "Quad. Hybrid QCN-19+ 1100 - 1925 MHz PSAS / OreSat 2019-11-06 v1 E.M. KJ7AOG"
Changed lines of the file:
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@@
 <text x="8.6" y="15" size="1.2" layer="21" font="vector" ratio="15" rot="SR180">P2</text>
 <text x="15" y="11.5" size="1.2" layer="21" font="vector" ratio="15" rot="R90">P1</text>
-<text x="10" y="12.6" size="1" layer="22" font="vector" ratio="15" rot="MR0" align="top-center">Quad. Hybrid QCN-19+
-1100 - 1925 MHz
+<text x="10" y="12.4" size="1" layer="22" font="vector" ratio="15" rot="MR0" align="top-center">Quad. Hybrid QCN-XXX+
 PSAS / OreSat
 2019-11-06 v1
