File: eagle/amp-LNA-BFPxxxF.brd (EAGLE design)
At the start: 26 x 20 mm, 21 parts, among them J1 142-0701-851, J2 142-0701-851, Q1 BFP740F

Commit message: Update current BFPxxxF
Parts:
- Q1: value BFP740F -> BFPXXXF
Changed lines of the file:
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@@
 <drawing>
 <settings>
-<setting alwaysvectorfont="yes"/>
+<setting alwaysvectorfont="no"/>
 <setting verticaltext="up"/>
 </settings>
@@
 <attribute name="NAME" x="8.3" y="10.5" size="0.2" layer="33" ratio="15" align="center"/>
 </element>
-<element name="Q1" library="Q-Infineon-BFPXXX-RF-BJT" package="TSFP4" value="BFP740F" x="12" y="10" smashed="yes" rot="R270">
+<element name="Q1" library="Q-Infineon-BFPXXX-RF-BJT" package="TSFP4" value="BFPXXXF" x="12" y="10" smashed="yes" rot="R270">
 <attribute name="NAME" x="11.1" y="7.5" size="0.6" layer="25" font="vector" ratio="15"/>
 </element>
