File: eagle/amp-LNA-BGB741L7ESD.sch (EAGLE design)
At the start: 19 parts, among them J1 142-0701-851, J2 142-0701-851, Q1 PMOS, U1 BGB7XXL7ESD

Commit message: Update BGB741L7ESD
Parts:
- C1, C2: value 47p -> 22p
- L1, L2: value 56n -> 27n
- R2: value 27k / NP -> 47k; device oresat-rcl:R-US_0603-B-NOSILK -> oresat-rcl:R-US_0402-B-NOSILK
- R3: value 47k -> 27k / NP; device oresat-rcl:R-US_0402-B-NOSILK -> oresat-rcl:R-US_0603-B-NOSILK
- renumbered R5 to R4
Connections:
- net 2V7: now also R3.2; no longer R2.2
- net GND: now also R2.1; no longer R3.1
- net N$1: now also R2.2; no longer R3.2
- net N$5: now also R3.1; no longer R2.1
Other:
- note added: "Infineon LNA BGB741L7ESD"
- note added: "L band 2nd Stage / IF Stage -------------------------- Vce = ~2.5V Ic = 6mA Gain = 18 dB NF = 1.2 dB Unconditionally Stable -------------------------- U1 = BGB741L7ESD R3 = 22k R4 = 0 L1 = 22n L2 = 22n"
- note added: "UHF - L band LNA (used as preamp) -------------------------- Vce = ~2.5V Ic = 8.0mA Gain = 18.4 dB @ 1265MHz NF = 1.2 dB Unconditionally Stable -------------------------- U1 = BGB741L7ESD R3 = 10k R4 = 0 L1 = 27n L2 = 27n"
- note removed: "808 MHz Performance: ----------------------------- Icq = 6mA NF = 1.1 dB G_T = 18.5 dB OP1dB = 13.5 dBm OIP3 = 21.5 dBm ----------------------------- S11 = -17.9 dB S22 = -16.4 dB S21 = 18.5 dB S12 = -21.1 dB"
- note removed: "L Band LO Amp / Wide band LNA"
- note removed: "LO Amp: BGB741L7ESD"
- note removed: "Quiescent Current Notes: R2 = 27k for 6mA R2 open for 5.2mA"
- moved on the sheet: R2, R3
Changed lines of the file:
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@@
 <part name="FRAME2" library="frames" library_urn="urn:adsk.eagle:library:229" deviceset="FRAME_A_L" device=""/>
 <part name="GND28" library="supply1" library_urn="urn:adsk.eagle:library:371" deviceset="GND" device=""/>
-<part name="C2" library="oresat-rcl" deviceset="C-EU" device="0402-C-NOSILK" value="47p"/>
+<part name="C2" library="oresat-rcl" deviceset="C-EU" device="0402-C-NOSILK" value="22p"/>
 <part name="GND29" library="supply1" library_urn="urn:adsk.eagle:library:371" deviceset="GND" device=""/>
 <part name="GND30" library="supply1" library_urn="urn:adsk.eagle:library:371" deviceset="GND" device=""/>
-<part name="R2" library="oresat-rcl" deviceset="R-US_" device="0603-B-NOSILK" value="27k / NP"/>
+<part name="R3" library="oresat-rcl" deviceset="R-US_" device="0603-B-NOSILK" value="27k / NP"/>
 <part name="C5" library="oresat-rcl" deviceset="C-EU" device="0603-B-NOSILK" value="1u"/>
 <part name="C4" library="oresat-rcl" deviceset="C-EU" device="0603-B-NOSILK" value="NP"/>
@@
 <part name="J1" library="J-Cinch-142-0701-851-SMA-end-launch" deviceset="142-0701-851" device=""/>
 <part name="J2" library="J-Cinch-142-0701-851-SMA-end-launch" deviceset="142-0701-851" device=""/>
-<part name="L2" library="oresat-rcl" deviceset="L-US" device="0603-C-NOSILK" value="56n"/>
-<part name="C1" library="oresat-rcl" deviceset="C-EU" device="0402-C-NOSILK" value="47p"/>
-<part name="L1" library="oresat-rcl" deviceset="L-US" device="0603-C-NOSILK" value="56n"/>
+<part name="L2" library="oresat-rcl" deviceset="L-US" device="0603-C-NOSILK" value="27n"/>
+<part name="C1" library="oresat-rcl" deviceset="C-EU" device="0402-C-NOSILK" value="22p"/>
+<part name="L1" library="oresat-rcl" deviceset="L-US" device="0603-C-NOSILK" value="27n"/>
 <part name="GND5" library="supply1" library_urn="urn:adsk.eagle:library:371" deviceset="GND" device=""/>
 <part name="GND7" library="supply1" library_urn="urn:adsk.eagle:library:371" deviceset="GND" device=""/>
@@
 <part name="JP2" library="pinhead" library_urn="urn:adsk.eagle:library:325" deviceset="PINHD-1X2" device="" package3d_urn="urn:adsk.eagle:package:22435/2"/>
 <part name="GND1" library="supply1" library_urn="urn:adsk.eagle:library:371" deviceset="GND" device=""/>
-<part name="R3" library="oresat-rcl" deviceset="R-US_" device="0402-B-NOSILK" value="47k"/>
+<part name="R2" library="oresat-rcl" deviceset="R-US_" device="0402-B-NOSILK" value="47k"/>
 <part name="GND3" library="supply1" library_urn="urn:adsk.eagle:library:371" deviceset="GND" device=""/>
 <part name="U1" library="U-Infineon-BGB7xxL7ESD-LNA" deviceset="BGB7XXL7ESD" device=""/>
-<part name="R5" library="oresat-rcl" deviceset="R-US_" device="0603-B-NOSILK" value="0"/>
+<part name="R4" library="oresat-rcl" deviceset="R-US_" device="0603-B-NOSILK" value="0"/>
 <part name="GND2" library="supply1" library_urn="urn:adsk.eagle:library:371" deviceset="GND" device=""/>
 </parts>
@@
 <sheet>
 <plain>
-<text x="176.53" y="26.67" size="5.08" layer="94">LO Amp: BGB741L7ESD</text>
+<text x="176.53" y="26.67" size="5.08" layer="94">Infineon LNA BGB741L7ESD</text>
 <text x="265.43" y="6.35" size="3.81" layer="94">1</text>
 <text x="182.88" y="184.15" size="1.778" layer="97">2.7V
@@
 <text x="148.59" y="157.48" size="1.778" layer="97">2V7 flood layer 3</text>
 <text x="144.018" y="159.512" size="1.778" layer="97" rot="R90">2V7 Net</text>
-<text x="127" y="76.2" size="1.778" layer="97" align="top-left">808 MHz Performance:
------------------------------
-Icq = 6mA
-NF = 1.1 dB
-G_T = 18.5 dB
-OP1dB = 13.5 dBm
-OIP3 = 21.5 dBm
------------------------------
-S11 = -17.9 dB
-S22 = -16.4 dB
-S21 = 18.5 dB
-S12 = -21.1 dB</text>
-<text x="162.56" y="76.2" size="1.778" layer="97" align="top-left">Quiescent Current Notes:
-R2 = 27k for 6mA
-R2 open for 5.2mA</text>
-<text x="63.5" y="142.24" size="3.556" layer="95">L Band LO Amp / Wide band LNA</text>
+<text x="69.85" y="74.93" size="1.778" layer="97" align="top-left">L band 2nd Stage / IF Stage
+--------------------------
+Vce = ~2.5V
+Ic = 6mA
+Gain = 18 dB
+NF = 1.2 dB
+Unconditionally Stable
+--------------------------
+U1 = BGB741L7ESD
+R3 = 22k
+R4 = 0
+L1 = 22n
+L2 = 22n</text>
+<text x="118.11" y="74.93" size="1.778" layer="97" align="top-left">UHF - L band LNA (used as preamp)
+--------------------------
+Vce = ~2.5V
+Ic = 8.0mA
+Gain = 18.4 dB @ 1265MHz
+NF = 1.2 dB
+Unconditionally Stable
+--------------------------
+U1 = BGB741L7ESD
+R3 = 10k
+R4 = 0
+L1 = 27n
+L2 = 27n</text>
 </plain>
 <instances>
@@
 <attribute name="VALUE" x="81.28" y="86.36" size="1.778" layer="96" rot="MR0"/>
 </instance>
-<instance part="R2" gate="R" x="157.48" y="130.81" smashed="yes" rot="R90">
+<instance part="R3" gate="R" x="157.48" y="130.81" smashed="yes" rot="R90">
 <attribute name="NAME" x="155.9814" y="127" size="1.778" layer="95" rot="R90"/>
-<attribute name="VALUE" x="160.782" y="124.46" size="1.778" layer="96" rot="R90"/>
 </instance>
 <instance part="C5" gate="CE" x="195.58" y="118.11" smashed="yes">
@@
 <attribute name="VALUE" x="114.3" y="163.83" size="1.778" layer="96"/>
 </instance>
-<instance part="R3" gate="R" x="134.62" y="168.91" smashed="yes" rot="R90">
+<instance part="R2" gate="R" x="134.62" y="168.91" smashed="yes" rot="R90">
 <attribute name="NAME" x="133.1214" y="165.1" size="1.778" layer="95" rot="R90"/>
 <attribute name="VALUE" x="137.922" y="165.1" size="1.778" layer="96" rot="R90"/>
@@
 <attribute name="VALUE" x="147.32" y="86.36" size="1.778" layer="96"/>
 </instance>
-<instance part="R5" gate="R" x="167.64" y="130.81" smashed="yes" rot="R90">
+<instance part="R4" gate="R" x="167.64" y="130.81" smashed="yes" rot="R90">
 <attribute name="NAME" x="166.1414" y="127" size="1.778" layer="95" rot="R90"/>
 <attribute name="VALUE" x="170.942" y="127" size="1.778" layer="96" rot="R90"/>
@@
 </segment>
 <segment>
-<pinref part="R3" gate="R" pin="1"/>
+<pinref part="R2" gate="R" pin="1"/>
 <pinref part="GND3" gate="1" pin="GND"/>
 </segment>
@@
 <net name="N$1" class="0">
 <segment>
-<pinref part="R3" gate="R" pin="2"/>
+<pinref part="R2" gate="R" pin="2"/>
 <wire x1="134.62" y1="173.99" x2="134.62" y2="176.53" width="0.1524" layer="91"/>
 <pinref part="JP2" gate="G$1" pin="2"/>
@@
 <wire x1="154.94" y1="101.6" x2="162.56" y2="101.6" width="0.1524" layer="91"/>
 <wire x1="162.56" y1="101.6" x2="162.56" y2="137.16" width="0.1524" layer="91"/>
-<pinref part="R2" gate="R" pin="2"/>
+<pinref part="R3" gate="R" pin="2"/>
 <wire x1="162.56" y1="137.16" x2="157.48" y2="137.16" width="0.1524" layer="91"/>
 <wire x1="157.48" y1="137.16" x2="157.48" y2="135.89" width="0.1524" layer="91"/>
-<pinref part="R5" gate="R" pin="2"/>
+<pinref part="R4" gate="R" pin="2"/>
 <wire x1="167.64" y1="135.89" x2="167.64" y2="137.16" width="0.1524" layer="91"/>
 <wire x1="167.64" y1="137.16" x2="162.56" y2="137.16" width="0.1524" layer="91"/>
@@
 <net name="N$5" class="0">
 <segment>
-<pinref part="R2" gate="R" pin="1"/>
+<pinref part="R3" gate="R" pin="1"/>
 <pinref part="U1" gate="G$1" pin="ADJ"/>
 <wire x1="157.48" y1="125.73" x2="157.48" y2="106.68" width="0.1524" layer="91"/>
@@
 <pinref part="C3" gate="CE" pin="1"/>
 <wire x1="177.8" y1="120.65" x2="177.8" y2="121.92" width="0.1524" layer="91"/>
-<pinref part="R5" gate="R" pin="1"/>
+<pinref part="R4" gate="R" pin="1"/>
 <pinref part="L2" gate="L" pin="1"/>
 <wire x1="167.64" y1="125.73" x2="167.64" y2="121.92" width="0.1524" layer="91"/>
