File: eagle/lpf-5th-order.sch (EAGLE design)
At the start: 7 parts, among them J1 142-0701-851, J2 142-0701-851

Commit message: Update values
Other:
- note added: "Inductors: Coilcraft 0402HP"
- note added: "L band (transmitter only) ------------------------------ L1, L2 = 5.1n C1, C3 = 4.7p C2 = 6.8p"
- note added: "UHF / IF (L band) ------------------------------ L1, L2 = 15.0n C1, C3 = 12.0p C2 = 18.0p"
Changed lines of the file:
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@@
 <text x="176.53" y="26.67" size="5.08" layer="94">5th Order Low-pass Filter</text>
 <text x="265.43" y="6.35" size="3.81" layer="94">1</text>
+<text x="154.94" y="88.9" size="1.778" layer="97" align="top-left">L band (transmitter only)
+------------------------------
+L1, L2 = 5.1n
+C1, C3 = 4.7p
+C2 = 6.8p
+</text>
+<text x="104.14" y="88.9" size="1.778" layer="97" align="top-left">UHF / IF (L band)
+------------------------------
+L1, L2 = 15.0n
+C1, C3 = 12.0p
+C2 = 18.0p
+</text>
+<text x="124.46" y="128.27" size="1.778" layer="97">Inductors: Coilcraft 0402HP</text>
 </plain>
 <instances>
@@
 </drawing>
 <compatibility>
+<note version="6.3" minversion="6.2.2" severity="warning">
+Since Version 6.2.2 text objects can contain more than one line,
+which will not be processed correctly with this version.
+</note>
 <note version="8.2" severity="warning">
 Since Version 8.2, EAGLE supports online libraries. The ids
