File: eagle/amp-LNA-BFPxxxF.sch (EAGLE design)
At the start: 21 parts, among them J1 142-0701-851, J2 142-0701-851, Q1 BFP740F

Commit message: Update current BFPxxxF
Parts:
- Q1: value BFP740F -> BFPXXXF
Other:
- note added: "L band 1st Stage - BFP740F -------------------------- Vce = 2.0V Ic = 10mA Gain = 22 dB NF = 0.66 dB Conditionally Stable -------------------------- Q1 = BFP740F R1 = 39 R2 = 27 R3 = 45.3k C1 = 22p C2 = 22p C7 = DNP L1 = 2.0n L2 >= 47n, <= 100n L3 = 10n L4 = 0 ohm R4 = 220"
- note added: "VHF - S band LNA - BFP843F (used as preamp) -------------------------- Vce = 1.5V Ic = 15mA Gain = 21.9 dB @ 1265MHz NF = 1.0 dB Unconditionally Stable -------------------------- Q1 = BFP843F R1 = 39 R2 = 39 R3 = 22k C1 = 100p C2 = 100p C7 = 560p L1 = 0 ohm L2 = 91n L3 = 91n L4 = 0 ohm R4 = open"
- note removed: "L band 740F Notes -------------------------- Vce = 2.0V Ic = 10mA Gain = 22 dB NF = 0.63 dB Conditionally Stable -------------------------- Q1 = BFP740F R1 = 39 R2 = 27 R3 = 45.3k C1 = 22p C2 = 22p C7 = DNP L1 = 2.0n L2 >= 47n L3 = 10n L4 = 0 ohm R4 = 220"
Changed lines of the file:
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@@
 <part name="R2" library="oresat-rcl" deviceset="R-US_" device="0603-C-NOSILK"/>
 <part name="GND2" library="supply1" library_urn="urn:adsk.eagle:library:371" deviceset="GND" device=""/>
-<part name="Q1" library="Q-Infineon-BFPXXX-RF-BJT" deviceset="BFPXXXF" device="" value="BFP740F"/>
+<part name="Q1" library="Q-Infineon-BFPXXX-RF-BJT" deviceset="BFPXXXF" device="" value="BFPXXXF"/>
 <part name="C7" library="oresat-rcl" deviceset="C-EU" device="0402-B-NOSILK"/>
 <part name="GND6" library="supply1" library_urn="urn:adsk.eagle:library:371" deviceset="GND" device=""/>
@@
 <text x="157.48" y="194.31" size="1.778" layer="97">2.7V
 External</text>
-<text x="85.09" y="72.39" size="1.778" layer="97" align="top-left">L band 740F Notes
+<text x="85.09" y="72.39" size="1.778" layer="97" align="top-left">L band 1st Stage - BFP740F
 --------------------------
 Vce = 2.0V
 Ic = 10mA
 Gain = 22 dB
-NF = 0.63 dB
+NF = 0.66 dB
 Conditionally Stable
 --------------------------
@@
 C7 = DNP
 L1 = 2.0n
-L2 &gt;= 47n
+L2 &gt;= 47n, &lt;= 100n
 L3 = 10n
 L4 = 0 ohm
@@
 <text x="140.97" y="82.55" size="1.778" layer="97">Emitter
 Degeneration</text>
+<text x="130.81" y="72.39" size="1.778" layer="97" align="top-left">VHF - S band LNA - BFP843F (used as preamp)
+--------------------------
+Vce = 1.5V
+Ic = 15mA
+Gain = 21.9 dB @ 1265MHz
+NF = 1.0 dB
+Unconditionally Stable
+--------------------------
+Q1 = BFP843F
+R1 = 39
+R2 = 39
+R3 = 22k
+C1 = 100p
+C2 = 100p
+C7 = 560p
+L1 = 0 ohm
+L2 = 91n
+L3 = 91n
+L4 = 0 ohm
+R4 = open</text>
 </plain>
 <instances>

Commit message: Update values
Other:
- note added: "L band 1st Stage - BFP740F -------------------------- Vce = 2.0V Ic = 10mA Gain = 22 dB NF = 0.66 dB Conditionally Stable -------------------------- Q1 = BFP740F R1 = 39 - 15 if using 2.5V LDO R2 = 27 R3 = 45.3k C1 = 22p C2 = 22p C7 = DNP L1 = 2.0n L2 >= 47n, <= 100n L3 = 10n L4 = 0 ohm R4 = 220"
- note added: "UHF LNA VHF - S band LNA - BFP843F (previously used as preamp) -------------------------- Vce = 1.5V Ic = 15mA Gain = 21.9 dB @ 1265MHz NF = 1.0 dB Unconditionally Stable -------------------------- Q1 = BFP843F R1 = 39 - 27 if using 2.5V LDO R2 = 39 R3 = 22k C1 = 100p C2 = 100p C7 = 560p L1 = 0 ohm L2 = 91n L3 = 91n L4 = 0 ohm R4 = open"
- note removed: "L band 1st Stage - BFP740F -------------------------- Vce = 2.0V Ic = 10mA Gain = 22 dB NF = 0.66 dB Conditionally Stable -------------------------- Q1 = BFP740F R1 = 39 R2 = 27 R3 = 45.3k C1 = 22p C2 = 22p C7 = DNP L1 = 2.0n L2 >= 47n, <= 100n L3 = 10n L4 = 0 ohm R4 = 220"
- note removed: "VHF - S band LNA - BFP843F (used as preamp) -------------------------- Vce = 1.5V Ic = 15mA Gain = 21.9 dB @ 1265MHz NF = 1.0 dB Unconditionally Stable -------------------------- Q1 = BFP843F R1 = 39 R2 = 39 R3 = 22k C1 = 100p C2 = 100p C7 = 560p L1 = 0 ohm L2 = 91n L3 = 91n L4 = 0 ohm R4 = open"
Changed lines of the file:
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@@
 <text x="157.48" y="194.31" size="1.778" layer="97">2.7V
 External</text>
-<text x="85.09" y="72.39" size="1.778" layer="97" align="top-left">L band 1st Stage - BFP740F
+<text x="67.31" y="72.39" size="1.778" layer="97" align="top-left">L band 1st Stage - BFP740F
 --------------------------
 Vce = 2.0V
@@
 --------------------------
 Q1 = BFP740F
-R1 = 39
+R1 = 39  -  15 if using 2.5V LDO
 R2 = 27
 R3 = 45.3k
@@
 <text x="140.97" y="82.55" size="1.778" layer="97">Emitter
 Degeneration</text>
-<text x="130.81" y="72.39" size="1.778" layer="97" align="top-left">VHF - S band LNA - BFP843F (used as preamp)
+<text x="130.81" y="72.39" size="1.778" layer="97" align="top-left">UHF LNA
+VHF - S band LNA - BFP843F (previously used as preamp)
 --------------------------
 Vce = 1.5V
@@
 --------------------------
 Q1 = BFP843F
-R1 = 39
+R1 = 39  -  27 if using 2.5V LDO
 R2 = 39
 R3 = 22k
