File: eagle/amp-PA-TQP7M9105-with-detect.brd (EAGLE design)
At the start: 44 x 34 mm, 46 parts, among them J1 142-0701-851, J2 142-0701-851, Q1 P-CH, Q2 N-CH, U1 TQP7M9105, U2 BDCN-20-13+, U3 LT5534, U4 LT5534

Commit message: Update PA TQP7M9105 values
Parts:
- C14: value 100n -> 47n
- C15: value 1n -> NP
- R7, R8: value 33k -> 47k
Changed lines of the file:
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@@
 <drawing>
 <settings>
-<setting alwaysvectorfont="yes"/>
+<setting alwaysvectorfont="no"/>
 <setting verticaltext="up"/>
 </settings>
@@
 <attribute name="NAME" x="26.5" y="8" size="0.3" layer="33" ratio="15" rot="R90" align="center"/>
 </element>
-<element name="R7" library="oresat-rcl" package=".0402-B-NOSILK" value="33k" x="4.2" y="25.6" smashed="yes">
+<element name="R7" library="oresat-rcl" package=".0402-B-NOSILK" value="47k" x="4.2" y="25.6" smashed="yes">
 <attribute name="NAME" x="3.6" y="24.15" size="0.8" layer="25" font="vector" ratio="15"/>
 <attribute name="NAME" x="4.2" y="25.6" size="0.2" layer="33" ratio="15" align="center"/>
@@
 <attribute name="VALUE" x="12.175" y="3.46" size="1.27" layer="27" rot="R90"/>
 </element>
-<element name="R8" library="oresat-rcl" package=".0402-B-NOSILK" value="33k" x="16" y="26.4" smashed="yes" rot="R180">
+<element name="R8" library="oresat-rcl" package=".0402-B-NOSILK" value="47k" x="16" y="26.4" smashed="yes" rot="R180">
 <attribute name="NAME" x="19" y="26.65" size="0.8" layer="25" font="vector" ratio="15" rot="R180"/>
 <attribute name="NAME" x="16" y="26.4" size="0.2" layer="33" ratio="15" rot="R180" align="center"/>
@@
 <attribute name="NAME" x="22.6" y="12.25" size="0.3" layer="33" ratio="15" align="center"/>
 </element>
-<element name="C14" library="oresat-rcl" package=".0603-B-NOSILK" value="100n" x="22.6" y="13.75" smashed="yes">
+<element name="C14" library="oresat-rcl" package=".0603-B-NOSILK" value="47n" x="22.6" y="13.75" smashed="yes">
 <attribute name="NAME" x="25" y="13.45" size="0.8" layer="25" font="vector" ratio="15"/>
 <attribute name="NAME" x="22.6" y="13.75" size="0.3" layer="33" ratio="15" align="center"/>
 </element>
-<element name="C15" library="oresat-rcl" package=".0603-B-NOSILK" value="1n" x="19.6" y="13.75" smashed="yes" rot="R180">
+<element name="C15" library="oresat-rcl" package=".0603-B-NOSILK" value="NP" x="19.6" y="13.75" smashed="yes" rot="R180">
 <attribute name="NAME" x="15.6" y="13.45" size="0.8" layer="25" font="vector" ratio="15"/>
 <attribute name="NAME" x="19.6" y="13.75" size="0.3" layer="33" ratio="15" rot="R180" align="center"/>
