File: eagle/test/TRL-calibration-thru-reflect-match.sch (EAGLE design)
At the start: 6 parts, among them J1 142-0701-851, J2 142-0701-851, J3 142-0701-851, J4 142-0701-851

Commit message: Update TRL-cal notes
Other:
- note added: "Note: For TRL the microstrip-38 can be used for the LINE standard with line length of 40 mm and velocity factor of 0.61; delay of 219ps."
- note added: "TRM Calibration Kit"
- note removed: "TRL Calibration Kit"
Changed lines of the file:
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@@
 <?xml version="1.0" encoding="utf-8"?>
 <!DOCTYPE eagle SYSTEM "eagle.dtd">
-<eagle version="9.2.2">
+<eagle version="9.5.1">
 <drawing>
 <settings>
@@
 <sheet>
 <plain>
-<text x="176.53" y="26.67" size="5.08" layer="94">TRL Calibration Kit</text>
+<text x="176.53" y="26.67" size="5.08" layer="94">TRM Calibration Kit</text>
 <text x="265.43" y="6.35" size="3.81" layer="94">1</text>
+<text x="81.28" y="58.42" size="1.778" layer="97">Note:  For TRL the microstrip-38 can be used for the LINE standard
+with line length of 40 mm and velocity factor of 0.61; delay of 219ps.</text>
 </plain>
 <instances>
@@
 </drawing>
 <compatibility>
+<note version="6.3" minversion="6.2.2" severity="warning">
+Since Version 6.2.2 text objects can contain more than one line,
+which will not be processed correctly with this version.
+</note>
 <note version="8.2" severity="warning">
 Since Version 8.2, EAGLE supports online libraries. The ids
