File: KiCad/_restore_backup_2026-05-20T06-30-41-497/amp-PA-GRF5504-with-detect.kicad_pcb (KiCad board)
At the start: 4 copper layers, 44 x 34 mm, 51 parts, among them J1 142-0701-851, J2 142-0701-851, Q1 P-CH, Q2 N-CH, U2 BDCN-20-13+, U3 LT5534, U4 LT5534, U5 GRF5504

Commit message: mess
Parts:
- J1, J2: value 142-0701-851 -> (none)
- U2: value BDCN-20-13+ -> (none)
Connections:
- J1 pad GND1: (no net) -> GND
- J1 pad GND2: (no net) -> GND
- J1 pad GND3: (no net) -> GND
- J2 pad GND1: (no net) -> GND
- J2 pad GND2: (no net) -> GND
- J2 pad GND3: (no net) -> GND
