File: KiCad/_restore_backup_2026-05-20T06-30-41-497/amp-PA-GRF5504-with-detect.kicad_sch (KiCad schematic)
At the start: 51 parts, among them J1 142-0701-851, J2 142-0701-851, J3 Conn_01x02, J4 Conn_01x02, Q1 P-CH, Q2 N-CH, U2 BDCN-20-13+, U3 LT5534, U4 LT5534, U5 GRF5504

Commit message: mess
Parts:
- D1: value GRN -> GREEN; footprint (none) -> oresat-diodes:LED-0603; symbol Device:LED_Filled -> amp-PA-TQP7M9105-with-detect-eagle-import:LED-GREEN0603
- JP3: renamed from J3; value Conn_01x02 -> PINHD-1X2; footprint (none) -> amp-PA-TQP7M9105-with-detect:1X02_325; symbol Connector_Generic:Conn_01x02 -> amp-PA-TQP7M9105-with-detect-eagle-import:PINHD-1X2
- JP4: renamed from J4; value Conn_01x02 -> PINHD-1X2; footprint (none) -> amp-PA-TQP7M9105-with-detect:1X02_325; symbol Connector_Generic:Conn_01x02 -> amp-PA-TQP7M9105-with-detect-eagle-import:PINHD-1X2
- Q1, Q2: footprint amp-PA-TQP7M9105-with-detect:SOT23_401 -> oresat-transistors:SOT23-6
- U5: footprint QFN-16_3MM_GRF -> oresat-ics:QFN-16_3MM_GRF
Connections:
- net GND: now also D1.C; no longer D1.1 (K)
- net at R1.1: now also D1.A; no longer D1.2 (A)
- net +3.3V renamed +3V3
